File: Adaptador/Eagle/adaptador_mcp3002_fpga.brd (EAGLE design)
At the start: 100.6 x 79.4 mm, 3 parts, among them IC1 MCP3202P

Commit message: Canviada la placa feta amb Eagle, ara els components estan com toca
Parts:
- moved SV1 30.5 mm to (15.2, 34.3)
- moved SV2 23.0 mm to (40.8, 34.3)
- moved IC1 1.52 mm to (29.0, 34.3), flipped to the top
Connections:
- net /CS: now also SV1.1; no longer SV1.2
- net CLK: now also SV1.7; no longer SV1.8
- net MISO: now also SV1.5; no longer SV1.6
- net MOSI: now also SV1.3; no longer SV1.4
Routing:
- net SENS: track 20.9 -> 28.0 mm
- net 3V3: track 44.8 -> 47.8 mm
- net MOSI: track 27.0 -> 29.0 mm
- net MISO: track 25.6 -> 27.4 mm
- net /CS: track 14.7 -> 16.0 mm
- net CLK: track 24.9 -> 24.4 mm
- added copper zone on layer 16, net GND
- removed copper zone on layer 1, net GND
Other:
- board text added: "+"
- board text added: "-"
- board text added: "IC1"
- board text added: "S"
- board text added: "SDAV 2016 Peshevski"
- board text added: "SV1"
- board text added: "SV2"
